File: Hardware/Magnetsteuerung_v2.0/Magnetsteuerung_v2.0.kicad_pcb (KiCad board)
At the start: 2 copper layers, 92.1 x 100.1 mm, 248 parts, among them J1 Conn_02x08_Odd_Even, J10 OUT1, J11 OUT1, J12 OUT1, J13 OUT1, J14 OUT1, J15 OUT1, J16 OUT1, J17 OUT1, J18 OUT1, J19 OUT1, J2 OUT1, J20 OUT1, J21 OUT1, J3 OUT1, J4 OUT1, J5 OUT1, J6 OUT1, J7 OUT1, J8 OUT1, J9 OUT1, Q1 Q_NMOS_GSD, Q10 Q_NMOS_GSD, Q11 Q_NMOS_GSD, Q12 Q_NMOS_GSD, Q13 Q_NMOS_GSD, Q14 Q_NMOS_GSD, Q15 Q_NMOS_GSD, Q16 Q_NMOS_GSD, Q17 Q_NMOS_GDS, Q2 Q_NMOS_GSD, Q3 Q_NMOS_GSD, Q4 Q_NMOS_GSD, Q5 Q_NMOS_GSD, Q6 Q_NMOS_GSD, Q7 Q_NMOS_GSD, Q8 Q_NMOS_GSD, U1 TL2575, U10 MCP1416R, U11 MCP1416R, U12 MCP1416R, U13 MCP1416R, U14 MCP1416R, U15 MCP1416R, U16 MCP1416R, U17 MCP1416R, U2 MCP1416R, U3 MCP1416R, U4 MCP1416R, U5 MCP1416R, U6 MCP1416R, U7 MCP1416R, U8 MCP1416R, U9 MCP1416R

Commit message: update layout
Parts:
- removed C3: 330u, Capacitor_SMD:CP_Elec_8x10
- removed D1: 1N5819, Diode_SMD:D_SOD-123
- removed D50: PMEG6010CEH, MK_Footprints:D_SOD_128_2
- removed L1: 330u, MK_Footprints:L_Bourns_5050
- removed U1: TL2575, Package_TO_SOT_SMD:TO-263-5_TabPin3
- added J22: OUT1, MK_Footprints:SPTAF_2, F.Cu at (136.8, 49.0)
- C1: value 100n -> 330u; footprint Capacitor_SMD:C_1206_3216Metric -> Capacitor_SMD:CP_Elec_8x10
- C2: value 100u -> 330u; footprint Capacitor_SMD:CP_Elec_10x10 -> Capacitor_SMD:CP_Elec_8x10
- moved C2 18.4 mm to (134.5, 68.5)
- moved C1 8.40 mm to (134.5, 59.5), turned to 0 degrees
Connections:
- C1 pad 1: Net-(C1-Pad1) -> +12V
- C2 pad 1: Net-(C1-Pad1) -> +12V
Routing:
- net GND: track 159.2 -> 103.3 mm, vias 34 -> 32
- net +12V: track 145.5 -> 115.4 mm, vias 18 -> 30
- net Net-(D1-Pad1): track 21.7 -> 0.00 mm, vias 1 -> 0
- net Net-(C1-Pad1): track 14.7 -> 0.00 mm, vias 1 -> 0
- net +48V: track 187.6 -> 182.5 mm
