File: Hardware/Magnetsteuerung_v2.1/Magnetsteuerung_v2.1.kicad_pcb (KiCad board)
At the start: 2 copper layers, 92.1 x 100.1 mm, 194 parts, among them J1 Conn_02x08_Odd_Even, J2 OUT1, J3 Conn_01x16, J4 OUT1, J7 OUT1, J8 OUT1, J9 Conn_01x16, Q1 Q_NMOS_GSD, Q10 Q_NMOS_GSD, Q11 Q_NMOS_GSD, Q12 Q_NMOS_GSD, Q13 Q_NMOS_GSD, Q14 Q_NMOS_GSD, Q15 Q_NMOS_GSD, Q16 Q_NMOS_GSD, Q17 Q_NMOS_GDS, Q2 Q_NMOS_GSD, Q3 Q_NMOS_GSD, Q4 Q_NMOS_GSD, Q5 Q_NMOS_GSD, Q6 Q_NMOS_GSD, Q7 Q_NMOS_GSD, Q8 Q_NMOS_GSD, U1 TL2575, U10 MCP1416R, U11 MCP1416R, U12 MCP1416R, U13 MCP1416R, U14 MCP1416R, U15 MCP1416R, U16 MCP1416R, U17 MCP1416R, U2 MCP1416R, U3 MCP1416R, U4 MCP1416R, U5 MCP1416R, U6 MCP1416R, U7 MCP1416R, U8 MCP1416R, U9 MCP1416R

Commit message: update layout v1.2
Parts:
- J1: value Conn_02x08_Odd_Even -> SPS_Connector
- Q1, Q10, Q11, Q12, Q13, Q14, Q15, Q16, Q2, Q3, Q4, Q5, Q6, Q7, Q8: value Q_NMOS_GSD -> DMN10H220LK3
- Q17: value Q_NMOS_GDS -> DMN10H220LK3
Connections:
- net +12V renamed +15V
- J1 pad 17: (no net) -> Net-(J1-Pad17)
- J1 pad 19: (no net) -> Net-(J1-Pad19)
- U10 pad 1: (no net) -> Net-(U10-Pad1)
- U11 pad 1: (no net) -> Net-(U11-Pad1)
- U12 pad 1: (no net) -> Net-(U12-Pad1)
- U13 pad 1: (no net) -> Net-(U13-Pad1)
- U14 pad 1: (no net) -> Net-(U14-Pad1)
- U15 pad 1: (no net) -> Net-(U15-Pad1)
- U16 pad 1: (no net) -> Net-(U16-Pad1)
- U17 pad 1: (no net) -> Net-(U17-Pad1)
- U2 pad 1: (no net) -> Net-(U2-Pad1)
- U3 pad 1: (no net) -> Net-(U3-Pad1)
- U4 pad 1: (no net) -> Net-(U4-Pad1)
- U5 pad 1: (no net) -> Net-(U5-Pad1)
- U6 pad 1: (no net) -> Net-(U6-Pad1)
- U7 pad 1: (no net) -> Net-(U7-Pad1)
- U8 pad 1: (no net) -> Net-(U8-Pad1)
- U9 pad 1: (no net) -> Net-(U9-Pad1)
Routing:
- net +15V: track 116.5 -> 124.0 mm, vias 53 -> 39
