File: Hardware/Magnetsteuerung_v2.1/OUT_1-8.kicad_sch (KiCad schematic)
At the start: 88 parts, among them Q1 Q_NMOS_GSD, Q2 Q_NMOS_GSD, Q3 Q_NMOS_GSD, Q4 Q_NMOS_GSD, Q5 Q_NMOS_GSD, Q6 Q_NMOS_GSD, Q7 Q_NMOS_GSD, Q8 Q_NMOS_GSD, U2 MCP1416R, U3 MCP1416R, U4 MCP1416R, U5 MCP1416R, U6 MCP1416R, U7 MCP1416R, U8 MCP1416R, U9 MCP1416R

Commit message: Finalisierung
Parts:
- C13, C16, C18, C20, C22, C24, C26, C8: Mouser Nr. (none) -> 187-CL10B105KA8NNNC
- C14, C17, C19, C21, C23, C25, C27, C9: Mouser Nr. (none) -> 710-885382206004
- C44, C45, C46, C47, C48, C49, C50, C51: Mouser Nr. (none) -> 187-CL32B106KMVNNWE
- D11, D12, D13, D2, D20, D21, D5, D6: Mouser Nr. (none) -> 710-150060VS55040
- D14, D15, D16, D22, D23, D4, D7, D8: Mouser Nr. (none) -> 771-PMEG6010CEH-QX
- R1, R13, R14, R15, R16, R17, R18, R2, R25, R26, R27, R28, R5, R6, R65, R66, R67, R68, R69, R7, R70, R71, R72, R8: Mouser Nr. (none) -> 71-RCG060310K0FKEA
- R10, R19, R20, R21, R29, R3, R30, R9: Hersteller Nr. RCG0603100RFKEA -> CRS0603AFX-1000ELF; Mouser Nr. (none) -> CRS0603AFX-1000ELF
- U2, U3, U4, U5, U6, U7, U8, U9: Mouser Nr. (none) -> 579-MCP1416RT-E/OT
