File: Hardware/Magnetsteuerung_v2.1/OUT_8-16.kicad_sch (KiCad schematic)
At the start: 88 parts, among them Q10 Q_NMOS_GSD, Q11 Q_NMOS_GSD, Q12 Q_NMOS_GSD, Q13 Q_NMOS_GSD, Q14 Q_NMOS_GSD, Q15 Q_NMOS_GSD, Q16 Q_NMOS_GSD, Q17 Q_NMOS_GSD, U10 MCP1416R, U11 MCP1416R, U12 MCP1416R, U13 MCP1416R, U14 MCP1416R, U15 MCP1416R, U16 MCP1416R, U17 MCP1416R

Commit message: Finalisierung
Parts:
- C10, C11, C12, C15, C4, C5, C6, C7: Mouser Nr. (none) -> 187-CL32B106KMVNNWE
- C28, C30, C32, C34, C36, C38, C40, C42: Mouser Nr. (none) -> 187-CL10B105KA8NNNC
- C29, C31, C33, C35, C37, C39, C41, C43: Mouser Nr. (none) -> 710-885382206004
- D26, D27, D28, D35, D36, D37, D44, D45: Mouser Nr. (none) -> 710-150060VS55040
- D29, D30, D31, D38, D39, D40, D46, D47: Mouser Nr. (none) -> 771-PMEG6010CEH-QX
- Q17: Mouser Nr. (none) -> 621-DMN10H220LK3-13
- R33, R34, R35, R36, R37, R38, R45, R46, R47, R48, R49, R50, R57, R58, R59, R60, R73, R74, R75, R76, R77, R78, R79, R80: Mouser Nr. (none) -> 71-RCG060310K0FKEA
- R39, R40, R41, R51, R52, R53, R61, R62: Hersteller Nr. RCG0603100RFKEA -> CRS0603AFX-1000ELF; Mouser Nr. (none) -> CRS0603AFX-1000ELF
- U10, U11, U12, U13, U14, U15, U16, U17: Mouser Nr. (none) -> 579-MCP1416RT-E/OT
